File: hw/kicad/kl24_breakout.kicad_pcb (KiCad board)
At the start: 2 copper layers, 23.4 x 20.8 mm, 37 parts, among them J1 USB-micro-ab, J2 ARM_10PIN, P1 TST, P10 TST, P11 TST, P12 TST, P13 TST, P14 TST, P17 TST, P18 TST, P20 TST, P21 TST, P22 TST, P23 TST, P24 TST, P25 TST, P26 TST, P27 TST, P28 TST, P29 TST, P30 TST, P31 TST, P32 TST, P33 5V, P34 GND, P9 TST, U1 MKL24Z64VFM4

Commit message: - layout
Parts:
- J2: moved to B.Cu
- turned J2 to 270 degrees
Routing:
- net N-000009: track 5.84 -> 0.00 mm
- net USB_DP: track 5.39 -> 0.00 mm
- net USB_DM: track 4.87 -> 0.00 mm
Changed lines of the file:
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@@
   (general
     (links 60)
-    (no_connects 55)
+    (no_connects 58)
     (area 96.5805 59.496 157.858333 82.812)
     (thickness 1.6)
-    (drawings 11)
-    (tracks 12)
+    (drawings 12)
+    (tracks 4)
     (zones 0)
     (modules 37)
@@
     )
   )
-  (module ARM_10_PIN_SMT (layer F.Cu)
-    (at 127 71.12 90)
-    (fp_text reference J2 (at -4.064 1.016 180) (layer F.SilkS)
-      (effects (font (size 1 1) (thickness 0.15)))
-    )
-    (fp_text value ARM_10PIN (at 0 4 90) (layer F.SilkS) hide
-      (effects (font (size 1 1) (thickness 0.15)))
-    )
-    (pad 1 smd oval (at -2.5 2.175 90) (size 0.76 1.75)
-      (layers F.Cu F.Paste F.Mask)
+  (module ARM_10_PIN_SMT (layer B.Cu)
+    (at 127 71.12 270)
+    (fp_text reference J2 (at -4.064 2.286 540) (layer B.SilkS)
+      (effects (font (size 1 1) (thickness 0.15)) (justify mirror))
+    )
+    (fp_text value ARM_10PIN (at 0 -4 270) (layer B.SilkS) hide
+      (effects (font (size 1 1) (thickness 0.15)) (justify mirror))
+    )
+    (pad 1 smd oval (at -2.5 -2.175 270) (size 0.76 1.75)
+      (layers B.Cu B.Paste B.Mask)
       (net 19 3.3V_SUPPLY)
     )
-    (pad 2 smd rect (at -2.5 -2.175 90) (size 0.76 1.75)
-      (layers F.Cu F.Paste F.Mask)
+    (pad 2 smd rect (at -2.5 2.175 270) (size 0.76 1.75)
+      (layers B.Cu B.Paste B.Mask)
       (net 5 13)
     )
-    (pad 3 smd rect (at -1.23 2.175 90) (size 0.76 1.75)
-      (layers F.Cu F.Paste F.Mask)
-      (net 24 GND)
-    )
-    (pad 4 smd rect (at -1.23 -2.175 90) (size 0.76 1.75)
-      (layers F.Cu F.Paste F.Mask)
+    (pad 3 smd rect (at -1.23 -2.175 270) (size 0.76 1.75)
+      (layers B.Cu B.Paste B.Mask)
+      (net 24 GND)
+    )
+    (pad 4 smd rect (at -1.23 2.175 270) (size 0.76 1.75)
+      (layers B.Cu B.Paste B.Mask)
       (net 2 10)
     )
-    (pad 5 smd rect (at 0.04 2.175 90) (size 0.76 1.75)
-      (layers F.Cu F.Paste F.Mask)
-      (net 24 GND)
-    )
-    (pad 6 smd rect (at 0.04 -2.175 90) (size 0.76 1.75)
-      (layers F.Cu F.Paste F.Mask)
-    )
-    (pad 7 smd rect (at 1.31 2.175 90) (size 0.76 1.75)
-      (layers F.Cu F.Paste F.Mask)
-      (net 24 GND)
-    )
-    (pad 8 smd rect (at 1.31 -2.175 90) (size 0.76 1.75)
-      (layers F.Cu F.Paste F.Mask)
-    )
-    (pad 9 smd rect (at 2.58 2.175 90) (size 0.76 1.75)
-      (layers F.Cu F.Paste F.Mask)
-      (net 24 GND)
-    )
-    (pad 10 smd rect (at 2.58 -2.175 90) (size 0.76 1.75)
-      (layers F.Cu F.Paste F.Mask)
+    (pad 5 smd rect (at 0.04 -2.175 270) (size 0.76 1.75)
+      (layers B.Cu B.Paste B.Mask)
+      (net 24 GND)
+    )
+    (pad 6 smd rect (at 0.04 2.175 270) (size 0.76 1.75)
+      (layers B.Cu B.Paste B.Mask)
+    )
+    (pad 7 smd rect (at 1.31 -2.175 270) (size 0.76 1.75)
+      (layers B.Cu B.Paste B.Mask)
+      (net 24 GND)
+    )
+    (pad 8 smd rect (at 1.31 2.175 270) (size 0.76 1.75)
+      (layers B.Cu B.Paste B.Mask)
+    )
+    (pad 9 smd rect (at 2.58 -2.175 270) (size 0.76 1.75)
+      (layers B.Cu B.Paste B.Mask)
+      (net 24 GND)
+    )
+    (pad 10 smd rect (at 2.58 2.175 270) (size 0.76 1.75)
+      (layers B.Cu B.Paste B.Mask)
       (net 33 nreset)
     )
+  )
+  (dimension 23.368 (width 0.25) (layer Cmts.User)
+    (gr_text "23.368 mm" (at 121.92 55.388001) (layer Cmts.User)
+      (effects (font (size 1 1) (thickness 0.25)))
+    )
+    (feature1 (pts (xy 133.604 62.23) (xy 133.604 54.388001)))
+    (feature2 (pts (xy 110.236 62.23) (xy 110.236 54.388001)))
+    (crossbar (pts (xy 110.236 56.388001) (xy 133.604 56.388001)))
+    (arrow1a (pts (xy 133.604 56.388001) (xy 132.477497 56.974421)))
+    (arrow1b (pts (xy 133.604 56.388001) (xy 132.477497 55.801581)))
+    (arrow2a (pts (xy 110.236 56.388001) (xy 111.362503 56.974421)))
+    (arrow2b (pts (xy 110.236 56.388001) (xy 111.362503 55.801581)))
+  )
+  (dimension 20.828 (width 0.25) (layer Cmts.User)
+    (gr_text "20.828 mm" (at 143.493998 71.12 270) (layer Cmts.User)
+      (effects (font (size 1 1) (thickness 0.25)))
+    )
+    (feature1 (pts (xy 131.318 81.534) (xy 144.493998 81.534)))
+    (feature2 (pts (xy 131.318 60.706) (xy 144.493998 60.706)))
+    (crossbar (pts (xy 142.493998 60.706) (xy 142.493998 81.534)))
+    (arrow1a (pts (xy 142.493998 81.534) (xy 141.907578 80.407497)))
+    (arrow1b (pts (xy 142.493998 81.534) (xy 143.080418 80.407497)))
+    (arrow2a (pts (xy 142.493998 60.706) (xy 141.907578 61.832503)))
+    (arrow2b (pts (xy 142.493998 60.706) (xy 143.080418 61.832503)))
   )
   (gr_line (start 110.236 62.23) (end 110.236 80.01) (angle 90) (layer Edge.Cuts) (width 0.15))
@@
     (effects (font (size 1 1) (thickness 0.25)))
   )
-  (dimension 20.701 (width 0.25) (layer Cmts.User)
-    (gr_text "20.701 mm" (at 153.399999 71.1835 270) (layer Cmts.User)
-      (effects (font (size 1 1) (thickness 0.25)))
-    )
-    (feature1 (pts (xy 150.114 81.534) (xy 154.399999 81.534)))
-    (feature2 (pts (xy 150.114 60.833) (xy 154.399999 60.833)))
-    (crossbar (pts (xy 152.399999 60.833) (xy 152.399999 81.534)))
-    (arrow1a (pts (xy 152.399999 81.534) (xy 151.813579 80.407497)))
-    (arrow1b (pts (xy 152.399999 81.534) (xy 152.986419 80.407497)))
-    (arrow2a (pts (xy 152.399999 60.833) (xy 151.813579 61.959503)))
-    (arrow2b (pts (xy 152.399999 60.833) (xy 152.986419 61.959503)))
-  )
   (gr_circle (center 125.5649 72.009) (end 125.7046 72.0471) (layer F.SilkS) (width 0.2))
-  (segment (start 117.475 66.548) (end 117.475 69.723) (width 0.254) (layer B.Cu) (net 29))
-  (segment (start 116.728 70.47) (end 117.475 69.723) (width 0.254) (layer B.Cu) (net 29))
-  (segment (start 116.728 70.47) (end 115.118 70.47) (width 0.254) (layer B.Cu) (net 29))
-  (segment (start 119.507 70.612) (end 118.349 71.77) (width 0.254) (layer B.Cu) (net 30))
-  (segment (start 118.349 71.77) (end 115.118 71.77) (width 0.254) (layer B.Cu) (net 30))
-  (segment (start 115.118 71.12) (end 117.602 71.12) (width 0.254) (layer B.Cu) (net 31))
-  (segment (start 118.491 70.231) (end 117.602 71.12) (width 0.254) (layer B.Cu) (net 31))
-  (segment (start 118.491 70.231) (end 118.491 68.58) (width 0.254) (layer B.Cu) (net 31))
   (segment (start 116.205 76.2) (end 115.118 76.2) (width 0.254) (layer B.Cu) (net 32))
   (segment (start 115.118 72.42) (end 115.118 76.2) (width 0.254) (layer B.Cu) (net 32))

Commit message: - save
Parts:
- moved C5 15.8 mm to (126.9, 75.9)
- moved R2 5.95 mm to (116.5, 75.2)
- moved R4 2.69 mm to (119.3, 65.7)
- moved R3 2.57 mm to (115.8, 65.7)
- moved D1 2.44 mm to (122.7, 65.7)
- moved R1 1.99 mm to (117.5, 67.7)
- moved JP1 1.57 mm to (126.1, 65.7), turned to 90 degrees
- moved U1 1.40 mm to (120.1, 71.1)
- moved C3 1.17 mm to (116.1, 77.0)
Routing:
- net 1: track 0.00 -> 10.5 mm
- net 12: track 0.00 -> 7.95 mm
- net N-000004: track 0.00 -> 7.84 mm, vias 0 -> 1
- net 9: track 0.00 -> 7.41 mm
- net 11: track 0.00 -> 7.00 mm
- net USB_DM: track 0.00 -> 5.27 mm
- net USB_VBUS: track 10.1 -> 15.2 mm, vias 0 -> 1
- net USB_DP: track 0.00 -> 4.65 mm
- net N-0000010: track 0.00 -> 2.72 mm, vias 0 -> 1
